File: hardware/gps-tracker.kicad_pcb (KiCad board)
At the start: 4 copper layers, 84.9 x 74.8 mm, 94 parts, among them J1 USB_B_Micro, J2 Conn_01x07, J3 Conn_01x08, J4 Conn_01x03, J5 Conn_01x04, J6 Conn_01x03, J7 Conn_01x02, SW1 SW_Push, SW2 SW_Push, SW3 SW_Push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

Commit message: Hardware revision v1.1:
- Switch to (hopefully) easier-to-solder light sensor
- Fix bootloader situation: use "One-click USB download of MCU" configuration from CH340 datasheet
- Connect radio reset line to MCU
- (Slightly) increase clearance for hand-soldering voltage regulators
Parts:
- added R9: 10k, Resistor_SMD:R_0402_1005Metric, B.Cu at (108.0, 115.8)
- U3: value LTR-303ALS-01 -> VEML7700-TT; footprint OptoDevice:Lite-On_LTR-303ALS-01 -> Homebrew:VISHAY_VEML7700-TT
- moved U3 4.49 mm to (89.0, 75.1), turned to 90 degrees
- moved C9 2.61 mm to (89.1, 77.7), turned to 0 degrees
- moved R22 2.54 mm to (79.4, 65.7)
- moved R13 1.70 mm to (113.0, 91.2)
- moved R10 1.70 mm to (114.7, 91.2)
- moved R4 0.41 mm to (108.3, 117.8), turned to -90 degrees
- moved C26 0.30 mm to (103.9, 103.3)
- moved D5 0.20 mm to (103.8, 100.9)
- moved C36 0.14 mm to (85.5, 63.6)
Connections:
- C1 pad 1: /~{DTR} -> /~{RTS}
- R10 pad 2: /SCL -> /SDA
- R13 pad 2: /SDA -> /SCL
- R4 pad 1: Net-(U2-~{CTS}) -> Net-(U2-TNOW)
- R4 pad 2: /~{DTR} -> GND
- U1 pad 3: unconnected-(U1-PC15-Pad3) -> /RADIO_RESETN
- U2 pad 4: /BOOT0 -> /~{RTS}
- U2 pad 5: Net-(U2-~{CTS}) -> unconnected-(U2-~{CTS}-Pad5)
- U2 pad 6: /~{DTR} -> Net-(U2-TNOW)
- U3 pad 1: VCC -> /SCL
- U3 pad 2: unconnected-(U3-NC-Pad2) -> VCC
- U3 pad 4: /SCL -> /SDA
- U7 pad 15: unconnected-(U7-NRST-Pad15) -> /RADIO_RESETN
Routing:
- net /RADIO_RESETN: track 0.00 -> 53.6 mm, vias 0 -> 4
- net /~{DTR}: track 19.0 -> 0.00 mm, vias 4 -> 0
- net GND: track 166.7 -> 185.4 mm, vias 15 -> 21
- net /~{RTS}: track 0.00 -> 9.51 mm
- net VCC: track 76.5 -> 82.5 mm
- net /SDA: track 50.6 -> 47.3 mm, vias 6 -> 5
- net /GPS_TX: track 56.5 -> 53.1 mm
- net Net-(U2-TNOW): track 0.00 -> 3.26 mm
- net /GPS_RX: track 48.1 -> 45.6 mm
- net /SCL: track 50.4 -> 48.0 mm
- net Net-(U9-EN): track 2.02 -> 4.28 mm
- net Net-(U2-~{CTS}): track 1.98 -> 0.00 mm
- net /BOOT0: track 55.4 -> 57.0 mm, vias 5 -> 4
- net /RADIO_BUSY: track 62.2 -> 61.1 mm
- net +BATT: track 108.2 -> 109.2 mm
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Other:
- board text added: "gps-tracker v1.1"
- board text removed: "gps-tracker v1.0"
