File: hardware/gps-tracker.kicad_sch (KiCad schematic)
At the start: 94 parts, among them J1 USB_B_Micro, J2 Conn_01x07, J3 Conn_01x08, J4 Conn_01x03, J5 Conn_01x04, J6 Conn_01x03, J7 Conn_01x02, SW1 SW_Push, SW2 SW_Push, SW3 SW_Push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

Commit message: Hardware revision v1.1:
- Switch to (hopefully) easier-to-solder light sensor
- Fix bootloader situation: use "One-click USB download of MCU" configuration from CH340 datasheet
- Connect radio reset line to MCU
- (Slightly) increase clearance for hand-soldering voltage regulators
Parts:
- removed U3: LTR-303ALS-01, OptoDevice:Lite-On_LTR-303ALS-01, symbol Sensor_Optical:LTR-303ALS-01
- added R9: 10k, Resistor_SMD:R_0402_1005Metric, symbol Device:R
- added U3: VEML7700-TT, Homebrew:VISHAY_VEML7700-TT, symbol Homebrew:VEML7700-TT
Connections:
- net BOOT0: now also R9.1; no longer U2.4 (~{RTS})
- net GND: now also R4.2, U3.3 (GND)
- net SCL: now also R13.2, U3.1 (SCL); no longer R10.2
- net SDA: now also R10.2, U3.4 (SDA); no longer R13.2
- net VCC: now also U3.2 (VDD)
- net RADIO_RESETN: now reaches U7.15 (NRST)
- net RADIO_RESETN: now also U1.3 (PC15)
- net at R4.1: now also U2.6 (TNOW), R9.2; no longer U2.5 (~{CTS})
- removed net ~{DTR}: C1.1, R4.2, U2.6 (TNOW)
- new net ~{RTS}: C1.1, U2.4 (~{RTS})
- no-connect marks 19 -> 17
Other:
- note added: ""One-click USB download of MCU" configuration"
- moved on the sheet: C9, R10, R13, R4
